Commit message: update ros2_control (feetech tmp)

File: auto_driver_description/urdf/auto_driver.urdf.xacro (robot description, xacro)
@@ -2,9 +2,9 @@
 <robot name="auto_driver" xmlns:xacro="http://ros.org/wiki/xacro">
   <xacro:include filename="$(find auto_driver_description)/urdf/auto_driver.xacro" />
-  <!-- <xacro:include filename="$(find auto_driver_description)/urdf/auto_driver.ros2_control.xacro" /> -->
+  <xacro:include filename="$(find auto_driver_description)/urdf/auto_driver.ros2_control.xacro" />
   <link name="world"/>
   <xacro:auto_driver parent="world">
     <origin xyz="0 0 0" rpy="0 0 0" />
   </xacro:auto_driver>
-  <!-- <xacro:auto_driver_ros2_control name="auto_driver_ros2_control" /> -->
+  <xacro:auto_driver_ros2_control name="auto_driver_ros2_control" />
 </robot>

File: auto_driver_description/urdf/auto_driver.xacro (robot description, xacro)
@@ -4,11 +4,11 @@
 <xacro:include filename="$(find auto_driver_description)/urdf/auto_driver.material.xacro" />
 <xacro:macro name="auto_driver" params="parent *origin">
-  <joint name="origin_to_link1" type="fixed">
+  <joint name="origin_to_base_frame" type="fixed">
     <xacro:insert_block name="origin" />
     <parent link="${parent}" />
-    <child link="link1" />
+    <child link="base_frame" />
     <axis xyz="0 0 1" />
   </joint>
-  <link name="link1">
+  <link name="base_frame">
     <visual>
       <origin xyz="0 0 0" rpy="0 -1.5708 0"/>
@@ -34,12 +34,12 @@
   <link name="fake_1_to_2" />
   <joint name="fake_1_to_2_joint" type="fixed">
-    <parent link="link1" />
+    <parent link="base_frame" />
     <child link="fake_1_to_2" />
-    <origin xyz="0 0 0.19" rpy="0 0 0" />
+    <origin xyz="-0.05 0 0.18" rpy="0 0 0" />
   </joint>
-  <joint name="yaw_joint" type="fixed">
+  <joint name="yaw_joint" type="revolute">
     <parent link="fake_1_to_2"/>
     <child link="yaw_link"/>
-    <origin xyz="0.0 0.0 0.005" rpy="0 0 -1.57079632679"/>
+    <origin xyz="0 0 0.005" rpy="0 0 0"/>
     <axis xyz="0 0 -1"/>
     <limit velocity="4.8" effort="1" lower="0.0" upper="2.0" />
@@ -72,5 +72,5 @@
     <parent link="yaw_link" />
     <child link="fake_2_to_3" />
-    <origin xyz="0 0 0" rpy="0 0 0" />
+    <origin xyz="0 0 0" rpy="-1.57079632679 0 0" />
   </joint>
   <link name="pitch_link">
@@ -96,9 +96,9 @@
     </inertial>
   </link>
-  <joint name="pitch_joint" type="fixed">
+  <joint name="pitch_joint" type="revolute">
     <parent link="fake_2_to_3"/>
     <child link="pitch_link"/>
     <origin xyz="0.0 0.0 0.005" rpy="0 0 0"/>
-    <axis xyz="0 0 -1"/>
+    <axis xyz="1 0 0"/>
     <limit velocity="4.8" effort="1" lower="0.0" upper="2.0" />
   </joint>

Commit message: Update auto2024.launch.py and package.xml***
***Update auto2024.launch.py to include new imports and parameters. Update package.xml to add new dependencies.

File: auto_driver_description/urdf/auto_driver.urdf.xacro (robot description, xacro)
@@ -2,9 +2,9 @@
 <robot name="auto_driver" xmlns:xacro="http://ros.org/wiki/xacro">
   <xacro:include filename="$(find auto_driver_description)/urdf/auto_driver.xacro" />
-  <xacro:include filename="$(find auto_driver_description)/urdf/auto_driver.ros2_control.xacro" />
+  <!-- <xacro:include filename="$(find auto_driver_description)/urdf/auto_driver.ros2_control.xacro" /> -->
   <link name="world"/>
   <xacro:auto_driver parent="world">
     <origin xyz="0 0 0" rpy="0 0 0" />
   </xacro:auto_driver>
-  <xacro:auto_driver_ros2_control name="auto_driver_ros2_control" />
+  <!-- <xacro:auto_driver_ros2_control name="auto_driver_ros2_control" /> -->
 </robot>

File: auto_driver_description/urdf/auto_driver.xacro (robot description, xacro)
@@ -36,5 +36,5 @@
     <parent link="base_frame" />
     <child link="fake_1_to_2" />
-    <origin xyz="0 0 0.18" rpy="0 0 0" />
+    <origin xyz="0 0 0.18" rpy="0 0 -1.57079632679" />
   </joint>
   <joint name="yaw_joint" type="revolute">
@@ -72,9 +72,9 @@
     <parent link="yaw_link" />
     <child link="fake_2_to_3" />
-    <origin xyz="0 0 0" rpy="-1.57079632679 0 0" />
+    <origin xyz="0 0 0.19" rpy="0 0 0" />
   </joint>
   <link name="pitch_link">
     <visual>
-      <origin xyz="0 0 0.019" rpy="0 0 0"/>
+      <origin xyz="0 0 -0.19" rpy="0 0 0"/>
       <geometry>
         <mesh filename="package://auto_driver_description/meshes/gimbal_pitch_link.stl" scale="0.001 0.001 0.001"/>
@@ -100,5 +100,5 @@
     <child link="pitch_link"/>
     <origin xyz="0.0 0.0 0.005" rpy="0 0 0"/>
-    <axis xyz="1 0 0"/>
+    <axis xyz="-1 0 0"/>
     <limit velocity="4.8" effort="1" lower="0.0" upper="2.0" />
   </joint>
