Commit message: fix urdf

File: auto_driver_description/urdf/auto_driver.xacro (robot description, xacro)
@@ -36,5 +36,5 @@
     <parent link="base_frame" />
     <child link="fake_1_to_2" />
-    <origin xyz="-0.05 0 0.18" rpy="0 0 0" />
+    <origin xyz="0 0 0.18" rpy="0 0 0" />
   </joint>
   <joint name="yaw_joint" type="revolute">
@@ -47,5 +47,5 @@
   <link name="yaw_link">
     <visual>
-      <origin xyz="0 0 0.019" rpy="0 0 0"/>
+      <origin xyz="0 -0.05 0.019" rpy="0 0 0"/>
       <geometry>
         <mesh filename="package://auto_driver_description/meshes/gimbal_yaw_link.stl" scale="0.001 0.001 0.001"/>
@@ -54,5 +54,5 @@
     </visual>
     <collision>
-      <origin xyz="0 0 0.019" rpy="0 0 0"/>
+      <origin xyz="0 -0.05 0.019" rpy="0 0 0"/>
       <geometry>
         <mesh filename="package://auto_driver_description/meshes/gimbal_yaw_link.stl" scale="0.001 0.001 0.001"/>

Commit message: Updated joint positions and added camera link

File: auto_driver_description/urdf/auto_driver.xacro (robot description, xacro)
@@ -72,5 +72,5 @@
     <parent link="yaw_link" />
     <child link="fake_2_to_3" />
-    <origin xyz="0 0 0.19" rpy="0 0 0" />
+    <origin xyz="0 -0.05 0.22" rpy="0 0 0" />
   </joint>
   <link name="pitch_link">
@@ -103,4 +103,10 @@
     <limit velocity="4.8" effort="1" lower="0.0" upper="2.0" />
   </joint>
+  <link name="camera_link" />
+  <joint name="pitch_joint_to_camera_link" type="fixed">
+    <parent link="pitch_link"/>
+    <child link="camera_link"/>
+    <origin xyz="-0.06 0.065 -0.08" rpy="0 0 1.57079632679" />
+  </joint>
 </xacro:macro>
 </robot>
